Commit message: Increased camera resolution and decreased camera pitch

File: src/sim/steve_description/urdf/steve.urdf (robot description, URDF)
Before this commit: robot steve, 15 links, 14 joints
Joints:
- joint joint_link_camera_support_link_camera_zed2i: origin xyz=0.02 0 0.065 rpy=0 0.4 0 -> xyz=0.02 0 0.065 rpy=0 0.3 0

Commit message: Changed urdf sensors

File: src/sim/steve_description/urdf/steve.urdf (robot description, URDF)
Before this commit: robot steve, 15 links, 14 joints
Joints:
- joint joint_link_camera_support_link_camera_zed2i: origin xyz=0.02 0 0.065 rpy=0 0.3 0 -> xyz=0.02 0 0.065 rpy=0 0.4 0
